Commit message: Experimentation with meshes and URDF generation

File: self_estimation/robot.urdf (robot description, URDF)
Before this commit: robot robot, 2 links, 1 joints
Links:
- link arm1: geometry collision mesh filename=Module_Arm(1).stl scale=0.1; visual mesh filename=Module_Arm(1).stl scale=0.1
Joints:
- joint joint1: origin xyz=0.0 0.34 0.0 -> xyz=0.0 0.34 0
