Commit message: started working on URDF generation via python

File: self_estimation/Starfish.urdf (robot description, URDF)
Before this commit: robot robot, 5 links, 4 joints
Links:
- added link arm3; collision box size=.68 .67 .3; visual box size=.68 .67 .3
- added link arm4; collision box size=.68 .67 .3; visual box size=.68 .67 .3
- added link body3; collision box size=.67 .688 .3; visual box size=.67 .688 .3
- added link body4; collision box size=.67 .688 .3; visual box size=.67 .688 .3
Joints:
- added joint joint5: type fixed, parent base_link, child body3, origin xyz=0.34 0 0, axis 0 1 0, limit lower=-1 upper=1.0 effort=0.0 velocity=0.0
- added joint joint6: type revolute, parent body3, child arm3, origin xyz=0.68 0 0, axis 0 1 0, limit lower=-1 upper=1.0 effort=0.0 velocity=0.0
- added joint joint7: type fixed, parent base_link, child body4, origin xyz=-0.34 0 0, axis 0 1 0, limit lower=-1 upper=1.0 effort=0.0 velocity=0.0
- added joint joint8: type revolute, parent body4, child arm4, origin xyz=-0.68 0 0, axis 0 1 0, limit lower=-1 upper=1.0 effort=0.0 velocity=0.0

File: self_estimation/robotTest.urdf (robot description, URDF)
Before this commit: robot test, 1 links, 0 joints
Links:
- removed link link1
- added link base_link, mass 1.0; collision box size=0.67 0.67 0.3; visual box size=0.67 0.67 0.3
- added link test, mass 1.0; collision box size=0.67 0.67 0.3; visual box size=0.68 0.67 0.3
Joints:
- added joint name: type revolute, parent base_link, child test, origin xyz=0.0 1.0 0.0 rpy=0.0 0.0 0.0, axis 1. 0. 0., limit lower=-1.0 upper=1.0 effort=1.0 velocity=1.0
