Commit message: work on basic generation

File: self_estimation/robotTest.urdf (robot description, URDF)
Before this commit: robot test, 2 links, 1 joints
Links:
- link test: geometry collision box size=0.67 0.67 0.3; visual box size=0.67 0.67 0.3
Joints:
- joint name: origin xyz=0.0 1.0 0.0 rpy=0.0 0.0 0.0 -> xyz=0.0 0.34 0.0 rpy=0.0 0.0 0.0
