Commit message: Added permuation simulation

File: self_estimation/Model_Permutation7_BestForArm_4.urdf (robot description, URDF)
Before this commit: robot Model_834, 9 links, 8 joints
Links:
- removed link arm_2_arm1
- removed link arm_2_arm2
- added link arm_Permutation_7_arm1, mass 1.0; collision box size=0.67 0.67 0.3; visual box size=0.67 0.67 0.3
- added link arm_Permutation_7_arm2, mass 1.0; collision box size=0.67 0.67 0.3; visual box size=0.67 0.67 0.3
Joints:
- removed joint arm_2_joint1
- removed joint arm_2_jointBase
- added joint arm_Permutation_7_joint1: type revolute, parent arm_Permutation_7_arm1, child arm_Permutation_7_arm2, origin xyz=0.0 0.68 0.0 rpy=0.0 0.0 0.0, axis 1. 0. 0., limit lower=-1.57 upper=1.57 effort=1.57 velocity=1.57
- added joint arm_Permutation_7_jointBase: type fixed, parent base_link, child arm_Permutation_7_arm1, origin xyz=0.34 0.34 0.0 rpy=0.0 0.0 -1.22, axis 1. 0. 0., limit lower=-1.57 upper=1.57 effort=1.57 velocity=1.57
- joint arm_0_jointBase: origin xyz=0.0 0.34 0.0 rpy=0.0 0.0 -0.02 -> xyz=0.0 0.34 0.0 rpy=0.0 0.0 0.48
- joint arm_1_jointBase: origin xyz=0.0 -0.34 0.0 rpy=0.0 0.0 2.41 -> xyz=0.0 -0.34 0.0 rpy=0.0 0.0 2.83
- joint arm_3_jointBase: origin xyz=-0.34 -0.34 0.0 rpy=0.0 0.0 0.83 -> xyz=-0.34 0.0 0.0 rpy=0.0 0.0 1.08
