Commit message: Pre large change commit

File: self_estimation/BestForArm_2.urdf (robot description, URDF)
Before this commit: robot Model_Models/Model_97.urdf7, 9 links, 8 joints
Links:
- removed link arm_1_arm1
- removed link arm_1_arm2
- removed link arm_Permutation_7_arm1
- removed link arm_Permutation_7_arm2
- added link arm_2_arm1, mass 1.0; collision box size=0.67 0.67 0.3; visual box size=0.67 0.67 0.3
- added link arm_2_arm2, mass 1.0; collision box size=0.67 0.67 0.3; visual box size=0.67 0.67 0.3
- added link arm_Permutation_41_arm1, mass 1.0; collision box size=0.67 0.67 0.3; visual box size=0.67 0.67 0.3
- added link arm_Permutation_41_arm2, mass 1.0; collision box size=0.67 0.67 0.3; visual box size=0.67 0.67 0.3
Joints:
- removed joint arm_1_joint1
- removed joint arm_1_jointBase
- removed joint arm_Permutation_7_joint1
- removed joint arm_Permutation_7_jointBase
- added joint arm_2_joint1: type revolute, parent arm_2_arm1, child arm_2_arm2, origin xyz=0.0 0.68 0.0 rpy=0.0 0.0 0.0, axis 1. 0. 0., limit lower=-1.57 upper=1.57 effort=1.57 velocity=1.57
- added joint arm_2_jointBase: type fixed, parent base_link, child arm_2_arm1, origin xyz=0.34 0.0 0.0 rpy=0.0 0.0 -1.5, axis 1. 0. 0., limit lower=-1.57 upper=1.57 effort=1.57 velocity=1.57
- added joint arm_Permutation_41_joint1: type revolute, parent arm_Permutation_41_arm1, child arm_Permutation_41_arm2, origin xyz=0.0 0.68 0.0 rpy=0.0 0.0 0.0, axis 1. 0. 0., limit lower=-1.57 upper=1.57 effort=1.57 velocity=1.57
- added joint arm_Permutation_41_jointBase: type fixed, parent base_link, child arm_Permutation_41_arm1, origin xyz=0.0 -0.34 0.0 rpy=0.0 0.0 -2.503185307179587, axis 1. 0. 0., limit lower=-1.57 upper=1.57 effort=1.57 velocity=1.57
- joint arm_0_jointBase: origin xyz=0.0 0.34 0.0 rpy=0.0 0.0 0.48 -> xyz=-0.34 0.34 0.0 rpy=0.0 0.0 -0.09999999999999998
- joint arm_3_jointBase: origin xyz=-0.34 0.0 0.0 rpy=0.0 0.0 1.08 -> xyz=-0.34 -0.34 0.0 rpy=0.0 0.0 0.75
