Commit message: started working on magnitude and longer legs

File: self_estimation/1BestForArm_2.urdf (robot description, URDF)
Before this commit: robot Model_Models/testPiece.urdf8, 5 links, 4 joints
Links:
- removed link arm_Permutation_8_arm1
- removed link arm_Permutation_8_arm2
- added link arm_Permutation_23_arm1, mass 1.0; collision box size=0.67 0.67 0.3; visual box size=0.67 0.67 0.3
- added link arm_Permutation_23_arm2, mass 1.0; collision box size=0.67 0.67 0.3; visual box size=0.67 0.67 0.3
- added link set2_arm1, mass 1.0; collision box size=0.67 0.67 0.3; visual box size=0.67 0.67 0.3
- added link set2_arm2, mass 1.0; collision box size=0.67 0.67 0.3; visual box size=0.67 0.67 0.3
- added link set3_arm1, mass 1.0; collision box size=0.67 0.67 0.3; visual box size=0.67 0.67 0.3
- added link set3_arm2, mass 1.0; collision box size=0.67 0.67 0.3; visual box size=0.67 0.67 0.3
Joints:
- removed joint arm_Permutation_8_joint1
- removed joint arm_Permutation_8_jointBase
- added joint arm_Permutation_23_joint1: type revolute, parent arm_Permutation_23_arm1, child arm_Permutation_23_arm2, origin xyz=0.0 0.68 0.0 rpy=0.0 0.0 0.0, axis 1. 0. 0., limit lower=-1.57 upper=1.57 effort=1.57 velocity=1.57
- added joint arm_Permutation_23_jointBase: type fixed, parent base_link, child arm_Permutation_23_arm1, origin xyz=0.0 -0.34 0.0 rpy=0.0 0.0 2.28, axis 1. 0. 0., limit lower=-1.57 upper=1.57 effort=1.57 velocity=1.57
- added joint set2_joint1: type revolute, parent set2_arm1, child set2_arm2, origin xyz=0.0 0.68 0.0 rpy=0.0 0.0 0.0, axis 1. 0. 0., limit lower=-1.57 upper=1.57 effort=1.57 velocity=1.57
- added joint set2_jointBase: type fixed, parent base_link, child set2_arm1, origin xyz=0.0 -0.34 0.0 rpy=0.0 0.0 -2.0821044779583477, axis 1. 0. 0., limit lower=-1.57 upper=1.57 effort=1.57 velocity=1.57
- added joint set3_joint1: type revolute, parent set3_arm1, child set3_arm2, origin xyz=0.0 0.68 0.0 rpy=0.0 0.0 0.0, axis 1. 0. 0., limit lower=-1.57 upper=1.57 effort=1.57 velocity=1.57
- added joint set3_jointBase: type fixed, parent base_link, child set3_arm1, origin xyz=-0.34 0.0 0.0 rpy=0.0 0.0 1.5709761334099326, axis 1. 0. 0., limit lower=-1.57 upper=1.57 effort=1.57 velocity=1.57
- joint set0_jointBase: origin xyz=0.0 0.34 0.0 rpy=0.0 0.0 0.0008016443998810793 -> xyz=0.0 0.34 0.0 rpy=0.0 0.0 0.0001448603526395746

File: self_estimation/1BestForArm_4.urdf (robot description, URDF)
Before this commit: robot Model_Models/testPiece.urdf94, 9 links, 8 joints
Links:
- removed link arm_Permutation_94_arm1
- removed link arm_Permutation_94_arm2
- removed link set2_arm1
- removed link set2_arm2
- added link arm_Permutation_90_arm1, mass 1.0; collision box size=0.67 0.67 0.3; visual box size=0.67 0.67 0.3
- added link arm_Permutation_90_arm2, mass 1.0; collision box size=0.67 0.67 0.3; visual box size=0.67 0.67 0.3
- added link set0_arm1, mass 1.0; collision box size=0.67 0.67 0.3; visual box size=0.67 0.67 0.3
- added link set0_arm2, mass 1.0; collision box size=0.67 0.67 0.3; visual box size=0.67 0.67 0.3
Joints:
- removed joint arm_Permutation_94_joint1
- removed joint arm_Permutation_94_jointBase
- removed joint set2_joint1
- removed joint set2_jointBase
- added joint arm_Permutation_90_joint1: type revolute, parent arm_Permutation_90_arm1, child arm_Permutation_90_arm2, origin xyz=0.0 0.68 0.0 rpy=0.0 0.0 0.0, axis 1. 0. 0., limit lower=-1.57 upper=1.57 effort=1.57 velocity=1.57
- added joint arm_Permutation_90_jointBase: type fixed, parent base_link, child arm_Permutation_90_arm1, origin xyz=0.34 -0.34 0.0 rpy=0.0 0.0 0.49, axis 1. 0. 0., limit lower=-1.57 upper=1.57 effort=1.57 velocity=1.57
- added joint set0_joint1: type revolute, parent set0_arm1, child set0_arm2, origin xyz=0.0 0.68 0.0 rpy=0.0 0.0 0.0, axis 1. 0. 0., limit lower=-1.57 upper=1.57 effort=1.57 velocity=1.57
- added joint set0_jointBase: type fixed, parent base_link, child set0_arm1, origin xyz=0.0 0.34 0.0 rpy=0.0 0.0 0.0001448603526395746, axis 1. 0. 0., limit lower=-1.57 upper=1.57 effort=1.57 velocity=1.57

File: self_estimation/1BestForArm_6.urdf (robot description, URDF)
Before this commit: robot Model_Models/Model_186.urdf60, 9 links, 8 joints
Links:
- removed link arm_0_arm1
- removed link arm_0_arm2
- removed link arm_1_arm1
- removed link arm_1_arm2
- removed link arm_2_arm1
- removed link arm_2_arm2
- removed link arm_Permutation_60_arm1
- removed link arm_Permutation_60_arm2
- added link arm_Permutation_17_arm1, mass 1.0; collision box size=0.67 0.67 0.3; visual box size=0.67 0.67 0.3
- added link arm_Permutation_17_arm2, mass 1.0; collision box size=0.67 0.67 0.3; visual box size=0.67 0.67 0.3
- added link set0_arm1, mass 1.0; collision box size=0.67 0.67 0.3; visual box size=0.67 0.67 0.3
- added link set0_arm2, mass 1.0; collision box size=0.67 0.67 0.3; visual box size=0.67 0.67 0.3
- added link set1_arm1, mass 1.0; collision box size=0.67 0.67 0.3; visual box size=0.67 0.67 0.3
- added link set1_arm2, mass 1.0; collision box size=0.67 0.67 0.3; visual box size=0.67 0.67 0.3
- added link set2_arm1, mass 1.0; collision box size=0.67 0.67 0.3; visual box size=0.67 0.67 0.3
- added link set2_arm2, mass 1.0; collision box size=0.67 0.67 0.3; visual box size=0.67 0.67 0.3
Joints:
- removed joint arm_0_joint1
- removed joint arm_0_jointBase
- removed joint arm_1_joint1
- removed joint arm_1_jointBase
- removed joint arm_2_joint1
- removed joint arm_2_jointBase
- removed joint arm_Permutation_60_joint1
- removed joint arm_Permutation_60_jointBase
- added joint arm_Permutation_17_joint1: type revolute, parent arm_Permutation_17_arm1, child arm_Permutation_17_arm2, origin xyz=0.0 0.68 0.0 rpy=0.0 0.0 0.0, axis 1. 0. 0., limit lower=-1.57 upper=1.57 effort=1.57 velocity=1.57
- added joint arm_Permutation_17_jointBase: type fixed, parent base_link, child arm_Permutation_17_arm1, origin xyz=-0.34 0.0 0.0 rpy=0.0 0.0 1.56, axis 1. 0. 0., limit lower=-1.57 upper=1.57 effort=1.57 velocity=1.57
- added joint set0_joint1: type revolute, parent set0_arm1, child set0_arm2, origin xyz=0.0 0.68 0.0 rpy=0.0 0.0 0.0, axis 1. 0. 0., limit lower=-1.57 upper=1.57 effort=1.57 velocity=1.57
- added joint set0_jointBase: type fixed, parent base_link, child set0_arm1, origin xyz=0.0 0.34 0.0 rpy=0.0 0.0 0.0001448603526395746, axis 1. 0. 0., limit lower=-1.57 upper=1.57 effort=1.57 velocity=1.57
- added joint set1_joint1: type revolute, parent set1_arm1, child set1_arm2, origin xyz=0.0 0.68 0.0 rpy=0.0 0.0 0.0, axis 1. 0. 0., limit lower=-1.57 upper=1.57 effort=1.57 velocity=1.57
- added joint set1_jointBase: type fixed, parent base_link, child set1_arm1, origin xyz=0.0 -0.34 0.0 rpy=0.0 0.0 3.141304589488269, axis 1. 0. 0., limit lower=-1.57 upper=1.57 effort=1.57 velocity=1.57
- added joint set2_joint1: type revolute, parent set2_arm1, child set2_arm2, origin xyz=0.0 0.68 0.0 rpy=0.0 0.0 0.0, axis 1. 0. 0., limit lower=-1.57 upper=1.57 effort=1.57 velocity=1.57
- added joint set2_jointBase: type fixed, parent base_link, child set2_arm1, origin xyz=0.0 -0.34 0.0 rpy=0.0 0.0 -2.0821044779583477, axis 1. 0. 0., limit lower=-1.57 upper=1.57 effort=1.57 velocity=1.57

File: self_estimation/Models/testPiece.urdf (robot description, URDF)
Before this commit: robot estimationBasic, 5 links, 4 joints
Links:
- added link set2_arm1, mass 1.0; collision box size=0.67 0.67 0.3; visual box size=0.67 0.67 0.3
- added link set2_arm2, mass 1.0; collision box size=0.67 0.67 0.3; visual box size=0.67 0.67 0.3
- added link set3_arm1, mass 1.0; collision box size=0.67 0.67 0.3; visual box size=0.67 0.67 0.3
- added link set3_arm2, mass 1.0; collision box size=0.67 0.67 0.3; visual box size=0.67 0.67 0.3
- added link set4_arm1, mass 1.0; collision box size=0.67 0.67 0.3; visual box size=0.67 0.67 0.3
- added link set4_arm2, mass 1.0; collision box size=0.67 0.67 0.3; visual box size=0.67 0.67 0.3
- added link set5_arm1, mass 1.0; collision box size=0.67 0.67 0.3; visual box size=0.67 0.67 0.3
- added link set5_arm2, mass 1.0; collision box size=0.67 0.67 0.3; visual box size=0.67 0.67 0.3
Joints:
- added joint set2_joint1: type revolute, parent set2_arm1, child set2_arm2, origin xyz=0.0 0.68 0.0 rpy=0.0 0.0 0.0, axis 1. 0. 0., limit lower=-1.57 upper=1.57 effort=1.57 velocity=1.57
- added joint set2_jointBase: type fixed, parent base_link, child set2_arm1, origin xyz=0.0 -0.34 0.0 rpy=0.0 0.0 1.7691421450193296, axis 1. 0. 0., limit lower=-1.57 upper=1.57 effort=1.57 velocity=1.57
- added joint set3_joint1: type revolute, parent set3_arm1, child set3_arm2, origin xyz=0.0 0.68 0.0 rpy=0.0 0.0 0.0, axis 1. 0. 0., limit lower=-1.57 upper=1.57 effort=1.57 velocity=1.57
- added joint set3_jointBase: type fixed, parent base_link, child set3_arm1, origin xyz=0.0 -0.34 0.0 rpy=0.0 0.0 3.141190661515593, axis 1. 0. 0., limit lower=-1.57 upper=1.57 effort=1.57 velocity=1.57
- added joint set4_joint1: type revolute, parent set4_arm1, child set4_arm2, origin xyz=0.0 0.68 0.0 rpy=0.0 0.0 0.0, axis 1. 0. 0., limit lower=-1.57 upper=1.57 effort=1.57 velocity=1.57
- added joint set4_jointBase: type fixed, parent base_link, child set4_arm1, origin xyz=0.0 -0.34 0.0 rpy=0.0 0.0 1.779909339039376, axis 1. 0. 0., limit lower=-1.57 upper=1.57 effort=1.57 velocity=1.57
- added joint set5_joint1: type revolute, parent set5_arm1, child set5_arm2, origin xyz=0.0 0.68 0.0 rpy=0.0 0.0 0.0, axis 1. 0. 0., limit lower=-1.57 upper=1.57 effort=1.57 velocity=1.57
- added joint set5_jointBase: type fixed, parent base_link, child set5_arm1, origin xyz=0.0 -0.34 0.0 rpy=0.0 0.0 -1.7799622275675964, axis 1. 0. 0., limit lower=-1.57 upper=1.57 effort=1.57 velocity=1.57
- joint set0_jointBase: origin xyz=0.0 0.34 0.0 rpy=0.0 0.0 0.0008016443998810793 -> xyz=0.0 0.34 0.0 rpy=0.0 0.0 -0.0005951622390284477
- joint set1_jointBase: origin xyz=-0.34 -0.34 0.0 rpy=0.0 0.0 -3.1414337214449355 -> xyz=0.0 0.34 0.0 rpy=0.0 0.0 -0.00033759424526136616

File: self_estimation/christanRobot.urdf (robot description, URDF)
Before this commit: robot Model_Models/Model_140.urdf41, 9 links, 8 joints
Links:
- removed link arm_0_arm1
- removed link arm_0_arm2
- removed link arm_2_arm1
- removed link arm_2_arm2
- removed link arm_3_arm1
- removed link arm_3_arm2
- removed link arm_Permutation_41_arm1
- removed link arm_Permutation_41_arm2
- added link set1_arm1, mass 1.0; collision box size=0.67 0.67 0.3; visual box size=0.67 0.67 0.3
- added link set1_arm2, mass 1.0; collision box size=0.67 0.67 0.3; visual box size=0.67 0.67 0.3
- added link set2_arm1, mass 1.0; collision box size=0.67 0.67 0.3; visual box size=0.67 0.67 0.3
- added link set2_arm2, mass 1.0; collision box size=0.67 0.67 0.3; visual box size=0.67 0.67 0.3
- added link set3_arm1, mass 1.0; collision box size=0.67 0.67 0.3; visual box size=0.67 0.67 0.3
- added link set3_arm2, mass 1.0; collision box size=0.67 0.67 0.3; visual box size=0.67 0.67 0.3
- added link set4_arm1, mass 1.0; collision box size=0.67 0.67 0.3; visual box size=0.67 0.67 0.3
- added link set4_arm2, mass 1.0; collision box size=0.67 0.67 0.3; visual box size=0.67 0.67 0.3
- added link set5_arm1, mass 1.0; collision box size=0.67 0.67 0.3; visual box size=0.67 0.67 0.3
- added link set5_arm2, mass 1.0; collision box size=0.67 0.67 0.3; visual box size=0.67 0.67 0.3
Joints:
- removed joint arm_0_joint1
- removed joint arm_0_jointBase
- removed joint arm_2_joint1
- removed joint arm_2_jointBase
- removed joint arm_3_joint1
- removed joint arm_3_jointBase
- removed joint arm_Permutation_41_joint1
- removed joint arm_Permutation_41_jointBase
- added joint set1_joint1: type revolute, parent set1_arm1, child set1_arm2, origin xyz=0.0 0.68 0.0 rpy=0.0 0.0 0.0, axis 1. 0. 0., limit lower=-1.57 upper=1.57 effort=1.57 velocity=1.57
- added joint set1_jointBase: type fixed, parent base_link, child set1_arm1, origin xyz=0.0 0.34 0.0 rpy=0.0 0.0 0.0, axis 1. 0. 0., limit lower=-1.57 upper=1.57 effort=1.57 velocity=1.57
- added joint set2_joint1: type revolute, parent set2_arm1, child set2_arm2, origin xyz=0.0 0.68 0.0 rpy=0.0 0.0 0.0, axis 1. 0. 0., limit lower=-1.57 upper=1.57 effort=1.57 velocity=1.57
- added joint set2_jointBase: type fixed, parent base_link, child set2_arm1, origin xyz=0.0 -0.34 0.0 rpy=0.0 0.0 3.141, axis 1. 0. 0., limit lower=-1.57 upper=1.57 effort=1.57 velocity=1.57
- added joint set3_joint1: type revolute, parent set3_arm1, child set3_arm2, origin xyz=0.0 0.68 0.0 rpy=0.0 0.0 0.0, axis 1. 0. 0., limit lower=-1.57 upper=1.57 effort=1.57 velocity=1.57
- added joint set3_jointBase: type fixed, parent set1_arm2, child set3_arm1, origin xyz=0.0 0.68 0.0 rpy=0.0 0.0 0.0, axis 1. 0. 0., limit lower=-1.57 upper=1.57 effort=1.57 velocity=1.57
- added joint set4_joint1: type revolute, parent set4_arm1, child set4_arm2, origin xyz=0.0 0.68 0.0 rpy=0.0 0.0 0.0, axis 1. 0. 0., limit lower=-1.57 upper=1.57 effort=1.57 velocity=1.57
- added joint set4_jointBase: type fixed, parent base_link, child set4_arm1, origin xyz=-0.34 0.0 0.0 rpy=0.0 0.0 1.57, axis 1. 0. 0., limit lower=-1.57 upper=1.57 effort=1.57 velocity=1.57
- added joint set5_joint1: type revolute, parent set5_arm1, child set5_arm2, origin xyz=0.0 0.68 0.0 rpy=0.0 0.0 0.0, axis 1. 0. 0., limit lower=-1.57 upper=1.57 effort=1.57 velocity=1.57
- added joint set5_jointBase: type fixed, parent base_link, child set5_arm1, origin xyz=0.34 0.0 0.0 rpy=0.0 0.0 -1.57, axis 1. 0. 0., limit lower=-1.57 upper=1.57 effort=1.57 velocity=1.57

File: self_estimation/christanRobotLONG.urdf (robot description, URDF)
Before this commit: robot Model_Models/testPiece.urdf94, 9 links, 8 joints
Links:
- removed link arm_Permutation_94_arm1
- removed link arm_Permutation_94_arm2
- added link set4_arm1, mass 1.0; collision box size=0.67 0.67 0.3; visual box size=0.67 0.67 0.3
- added link set4_arm2, mass 1.0; collision box size=0.67 0.67 0.3; visual box size=0.67 0.67 0.3
- added link set5_arm1, mass 1.0; collision box size=0.67 0.67 0.3; visual box size=0.67 0.67 0.3
- added link set5_arm2, mass 1.0; collision box size=0.67 0.67 0.3; visual box size=0.67 0.67 0.3
- added link set6_arm1, mass 1.0; collision box size=0.67 0.67 0.3; visual box size=0.67 0.67 0.3
- added link set6_arm2, mass 1.0; collision box size=0.67 0.67 0.3; visual box size=0.67 0.67 0.3
Joints:
- removed joint arm_Permutation_94_joint1
- removed joint arm_Permutation_94_jointBase
- added joint set4_joint1: type revolute, parent set4_arm1, child set4_arm2, origin xyz=0.0 0.68 0.0 rpy=0.0 0.0 0.0, axis 1. 0. 0., limit lower=-1.57 upper=1.57 effort=1.57 velocity=1.57
- added joint set4_jointBase: type fixed, parent base_link, child set4_arm1, origin xyz=-0.34 0.0 0.0 rpy=0.0 0.0 1.57, axis 1. 0. 0., limit lower=-1.57 upper=1.57 effort=1.57 velocity=1.57
- added joint set5_joint1: type revolute, parent set5_arm1, child set5_arm2, origin xyz=0.0 0.68 0.0 rpy=0.0 0.0 0.0, axis 1. 0. 0., limit lower=-1.57 upper=1.57 effort=1.57 velocity=1.57
- added joint set5_jointBase: type fixed, parent base_link, child set5_arm1, origin xyz=0.34 0.0 0.0 rpy=0.0 0.0 -1.57, axis 1. 0. 0., limit lower=-1.57 upper=1.57 effort=1.57 velocity=1.57
- added joint set6_joint1: type revolute, parent set6_arm1, child set6_arm2, origin xyz=0.0 0.68 0.0 rpy=0.0 0.0 0.0, axis 1. 0. 0., limit lower=-1.57 upper=1.57 effort=1.57 velocity=1.57
- added joint set6_jointBase: type fixed, parent set3_arm2, child set6_arm1, origin xyz=0.0 0.68 0.0 rpy=0.0 0.0 0.0, axis 1. 0. 0., limit lower=-1.57 upper=1.57 effort=1.57 velocity=1.57
- joint set1_jointBase: origin xyz=0.0 -0.34 0.0 rpy=0.0 0.0 3.141304589488269 -> xyz=0.0 0.34 0.0 rpy=0.0 0.0 0.0
- joint set2_jointBase: origin xyz=0.0 -0.34 0.0 rpy=0.0 0.0 -2.0821044779583477 -> xyz=0.0 -0.34 0.0 rpy=0.0 0.0 3.141
- joint set3_jointBase: origin xyz=-0.34 0.0 0.0 rpy=0.0 0.0 1.5709761334099326 -> xyz=0.0 0.68 0.0 rpy=0.0 0.0 0.0; parent base_link -> set1_arm2

File: self_estimation/longBoi.urdf (robot description, URDF)
Before this commit: robot Model_Models/testPiece.urdf94, 9 links, 8 joints
Links:
- removed link arm_Permutation_94_arm1
- removed link arm_Permutation_94_arm2
- added link set4_arm1, mass 1.0; collision box size=0.67 0.67 0.3; visual box size=0.67 0.67 0.3
- added link set4_arm2, mass 1.0; collision box size=0.67 0.67 0.3; visual box size=0.67 0.67 0.3
Joints:
- removed joint arm_Permutation_94_joint1
- removed joint arm_Permutation_94_jointBase
- added joint set4_joint1: type revolute, parent set4_arm1, child set4_arm2, origin xyz=0.0 0.68 0.0 rpy=0.0 0.0 0.0, axis 1. 0. 0., limit lower=-1.57 upper=1.57 effort=1.57 velocity=1.57
- added joint set4_jointBase: type fixed, parent base_link, child set4_arm1, origin xyz=-0.34 0.0 0.0 rpy=0.0 0.0 1.57, axis 1. 0. 0., limit lower=-1.57 upper=1.57 effort=1.57 velocity=1.57
- joint set1_jointBase: origin xyz=0.0 -0.34 0.0 rpy=0.0 0.0 3.141304589488269 -> xyz=0.0 0.34 0.0 rpy=0.0 0.0 0.0
- joint set2_jointBase: origin xyz=0.0 -0.34 0.0 rpy=0.0 0.0 -2.0821044779583477 -> xyz=0.0 -0.34 0.0 rpy=0.0 0.0 3.141
- joint set3_jointBase: origin xyz=-0.34 0.0 0.0 rpy=0.0 0.0 1.5709761334099326 -> xyz=0.0 0.68 0.0 rpy=0.0 0.0 0.0; parent base_link -> set1_arm2
