Commit message: added permutations to algo

File: self_estimation/1BestForArm_8.urdf (robot description, URDF)
Before this commit: robot Model_Models/testPiece.urdf94, 9 links, 8 joints
Links:
- removed link arm_Permutation_94_arm1
- removed link arm_Permutation_94_arm2
- added link arm_Permutation_5_arm1, mass 1.0; collision box size=0.67 0.67 0.3; visual box size=0.67 0.67 0.3
- added link arm_Permutation_5_arm2, mass 1.0; collision box size=0.67 0.67 0.3; visual box size=0.67 0.67 0.3
- added link set0_arm1, mass 1.0; collision box size=0.67 0.67 0.3; visual box size=0.67 0.67 0.3
- added link set0_arm2, mass 1.0; collision box size=0.67 0.67 0.3; visual box size=0.67 0.67 0.3
Joints:
- removed joint arm_Permutation_94_joint1
- removed joint arm_Permutation_94_jointBase
- added joint arm_Permutation_5_joint1: type revolute, parent arm_Permutation_5_arm1, child arm_Permutation_5_arm2, origin xyz=0.0 0.68 0.0 rpy=0.0 0.0 0.0, axis 1. 0. 0., limit lower=-1.57 upper=1.57 effort=1.57 velocity=1.57
- added joint arm_Permutation_5_jointBase: type fixed, parent base_link, child arm_Permutation_5_arm1, origin xyz=0.0 0.34 0.0 rpy=0.0 0.0 0.53, axis 1. 0. 0., limit lower=-1.57 upper=1.57 effort=1.57 velocity=1.57
- added joint set0_joint1: type revolute, parent set0_arm1, child set0_arm2, origin xyz=0.0 0.68 0.0 rpy=0.0 0.0 0.0, axis 1. 0. 0., limit lower=-1.57 upper=1.57 effort=1.57 velocity=1.57
- added joint set0_jointBase: type fixed, parent base_link, child set0_arm1, origin xyz=0.0 -0.34 0.0 rpy=0.0 0.0 3.140996777702981, axis 1. 0. 0., limit lower=-1.57 upper=1.57 effort=1.57 velocity=1.57
- joint set1_jointBase: origin xyz=0.0 -0.34 0.0 rpy=0.0 0.0 3.141304589488269 -> xyz=-0.34 0.34 0.0 rpy=0.0 0.0 0.9982080703103466
- joint set2_jointBase: origin xyz=0.0 -0.34 0.0 rpy=0.0 0.0 -2.0821044779583477 -> xyz=0.34 0.34 0.0 rpy=0.0 0.0 -1.0760221271669443
- joint set3_jointBase: origin xyz=-0.34 0.0 0.0 rpy=0.0 0.0 1.5709761334099326 -> xyz=0.34 0.34 0.0 rpy=0.0 0.0 -1.0006509717523158

File: self_estimation/Models/leaf.urdf (robot description, URDF)
Before this commit: robot Model_Models/testPiece.urdf17, 9 links, 8 joints
Links:
- removed link arm_Permutation_17_arm1
- removed link arm_Permutation_17_arm2
- removed link set0_arm1
- removed link set0_arm2
- removed link set1_arm1
- removed link set1_arm2
- added link set5_arm1, mass 1.0; collision box size=0.67 0.67 0.3; visual box size=0.67 0.67 0.3
- added link set5_arm2, mass 1.0; collision box size=0.67 0.67 0.3; visual box size=0.67 0.67 0.3
- added link set6_arm1, mass 1.0; collision box size=0.67 0.67 0.3; visual box size=0.67 0.67 0.3
- added link set6_arm2, mass 1.0; collision box size=0.67 0.67 0.3; visual box size=0.67 0.67 0.3
- added link set7_arm1, mass 1.0; collision box size=0.67 0.67 0.3; visual box size=0.67 0.67 0.3
- added link set7_arm2, mass 1.0; collision box size=0.67 0.67 0.3; visual box size=0.67 0.67 0.3
- added link set8_arm1, mass 1.0; collision box size=0.67 0.67 0.3; visual box size=0.67 0.67 0.3
- added link set8_arm2, mass 1.0; collision box size=0.67 0.67 0.3; visual box size=0.67 0.67 0.3
Joints:
- removed joint arm_Permutation_17_joint1
- removed joint arm_Permutation_17_jointBase
- removed joint set0_joint1
- removed joint set0_jointBase
- removed joint set1_joint1
- removed joint set1_jointBase
- added joint set5_joint1: type revolute, parent set5_arm1, child set5_arm2, origin xyz=0.0 0.68 0.0 rpy=0.0 0.0 0.0, axis 1. 0. 0., limit lower=-1.57 upper=1.57 effort=1.57 velocity=1.57
- added joint set5_jointBase: type fixed, parent base_link, child set5_arm1, origin xyz=-0.34 0.34 0.0 rpy=0.0 0.0 0.785, axis 1. 0. 0., limit lower=-1.57 upper=1.57 effort=1.57 velocity=1.57
- added joint set6_joint1: type revolute, parent set6_arm1, child set6_arm2, origin xyz=0.0 0.68 0.0 rpy=0.0 0.0 0.0, axis 1. 0. 0., limit lower=-1.57 upper=1.57 effort=1.57 velocity=1.57
- added joint set6_jointBase: type fixed, parent base_link, child set6_arm1, origin xyz=0.34 -0.34 0.0 rpy=0.0 0.0 -0.785, axis 1. 0. 0., limit lower=-1.57 upper=1.57 effort=1.57 velocity=1.57
- added joint set7_joint1: type revolute, parent set7_arm1, child set7_arm2, origin xyz=0.0 0.68 0.0 rpy=0.0 0.0 0.0, axis 1. 0. 0., limit lower=-1.57 upper=1.57 effort=1.57 velocity=1.57
- added joint set7_jointBase: type fixed, parent base_link, child set7_arm1, origin xyz=0.34 0.34 0.0 rpy=0.0 0.0 -0.785, axis 1. 0. 0., limit lower=-1.57 upper=1.57 effort=1.57 velocity=1.57
- added joint set8_joint1: type revolute, parent set8_arm1, child set8_arm2, origin xyz=0.0 0.68 0.0 rpy=0.0 0.0 0.0, axis 1. 0. 0., limit lower=-1.57 upper=1.57 effort=1.57 velocity=1.57
- added joint set8_jointBase: type fixed, parent base_link, child set8_arm1, origin xyz=-0.34 -0.34 0.0 rpy=0.0 0.0 0.785, axis 1. 0. 0., limit lower=-1.57 upper=1.57 effort=1.57 velocity=1.57
- joint set2_jointBase: origin xyz=0.0 -0.34 0.0 rpy=0.0 0.0 -2.0821044779583477 -> xyz=0.0 -0.34 0.0 rpy=0.0 0.0 3.141

File: self_estimation/Models/testPiece.urdf (robot description, URDF)
Before this commit: robot estimationBasic, 13 links, 12 joints
Links:
- removed link set5_arm1
- removed link set5_arm2
Joints:
- removed joint set5_joint1
- removed joint set5_jointBase
- joint set0_jointBase: origin xyz=0.0 0.34 0.0 rpy=0.0 0.0 -0.0005951622390284477 -> xyz=0.0 -0.34 0.0 rpy=0.0 0.0 3.140996777702981
- joint set1_jointBase: origin xyz=0.0 0.34 0.0 rpy=0.0 0.0 -0.00033759424526136616 -> xyz=-0.34 0.34 0.0 rpy=0.0 0.0 0.9982080703103466
- joint set2_jointBase: origin xyz=0.0 -0.34 0.0 rpy=0.0 0.0 1.7691421450193296 -> xyz=0.34 0.34 0.0 rpy=0.0 0.0 -1.0760221271669443
- joint set3_jointBase: origin xyz=0.0 -0.34 0.0 rpy=0.0 0.0 3.141190661515593 -> xyz=0.34 0.34 0.0 rpy=0.0 0.0 -1.0006509717523158
- joint set4_jointBase: origin xyz=0.0 -0.34 0.0 rpy=0.0 0.0 1.779909339039376 -> xyz=-0.34 0.34 0.0 rpy=0.0 0.0 1.0755915533719016
