Commit message: added experiment related code and bug fix

File: self_estimation/Models/Model_test.urdf (robot description, URDF)
Before this commit: robot Model_test, 3 links, 2 joints
Links:
- removed link TEST_arm1
- removed link TEST_arm2
- added link TEST1_arm1, mass 1.0; collision box size=0.67 0.67 0.3; visual box size=0.67 0.67 0.3
- added link TEST1_arm2, mass 1.0; collision box size=0.67 0.67 0.3; visual box size=0.67 0.67 0.3
- added link TEST2_arm1, mass 1.0; collision box size=0.67 0.67 0.3; visual box size=0.67 0.67 0.3
- added link TEST2_arm2, mass 1.0; collision box size=0.67 0.67 0.3; visual box size=0.67 0.67 0.3
- added link TEST3_arm1, mass 1.0; collision box size=0.67 0.67 0.3; visual box size=0.67 0.67 0.3
- added link TEST3_arm2, mass 1.0; collision box size=0.67 0.67 0.3; visual box size=0.67 0.67 0.3
- added link TEST4_arm1, mass 1.0; collision box size=0.67 0.67 0.3; visual box size=0.67 0.67 0.3
- added link TEST4_arm2, mass 1.0; collision box size=0.67 0.67 0.3; visual box size=0.67 0.67 0.3
Joints:
- removed joint TEST_joint1
- removed joint TEST_jointBase
- added joint TEST1_joint1: type revolute, parent TEST1_arm1, child TEST1_arm2, origin xyz=0.0 0.68 0.0 rpy=0.0 0.0 0.0, axis 1. 0. 0., limit lower=-1.0 upper=1.0 effort=1.0 velocity=1.0
- added joint TEST1_jointBase: type fixed, parent base_link, child TEST1_arm1, origin xyz=0.0 0.34 0.0 rpy=0.0 0.0 0.0, axis 1. 0. 0., limit lower=-1.0 upper=1.0 effort=1.0 velocity=1.0
- added joint TEST2_joint1: type revolute, parent TEST2_arm1, child TEST2_arm2, origin xyz=0.0 0.68 0.0 rpy=0.0 0.0 0.0, axis 1. 0. 0., limit lower=-1.0 upper=1.0 effort=1.0 velocity=1.0
- added joint TEST2_jointBase: type fixed, parent base_link, child TEST2_arm1, origin xyz=0.0 -0.34 0.0 rpy=0.0 0.0 3.141, axis 1. 0. 0., limit lower=-1.0 upper=1.0 effort=1.0 velocity=1.0
- added joint TEST3_joint1: type revolute, parent TEST3_arm1, child TEST3_arm2, origin xyz=0.0 0.68 0.0 rpy=0.0 0.0 0.0, axis 1. 0. 0., limit lower=-1.0 upper=1.0 effort=1.0 velocity=1.0
- added joint TEST3_jointBase: type fixed, parent base_link, child TEST3_arm1, origin xyz=0.34 0.0 0.0 rpy=0.0 0.0 -1.57, axis 1. 0. 0., limit lower=-1.0 upper=1.0 effort=1.0 velocity=1.0
- added joint TEST4_joint1: type revolute, parent TEST4_arm1, child TEST4_arm2, origin xyz=0.0 0.68 0.0 rpy=0.0 0.0 0.0, axis 1. 0. 0., limit lower=-1.0 upper=1.0 effort=1.0 velocity=1.0
- added joint TEST4_jointBase: type fixed, parent base_link, child TEST4_arm1, origin xyz=-0.34 0.0 0.0 rpy=0.0 0.0 1.57, axis 1. 0. 0., limit lower=-1.0 upper=1.0 effort=1.0 velocity=1.0

File: self_estimation/STARFISH2.0.urdf (robot description, URDF)
Before this commit: robot Model_0, 9 links, 8 joints
Links:
- removed link arm_0_arm1
- removed link arm_0_arm2
- removed link arm_1_arm1
- removed link arm_1_arm2
- removed link arm_2_arm1
- removed link arm_2_arm2
- removed link arm_3_arm1
- removed link arm_3_arm2
- added link set1_arm1, mass 1.0; collision box size=0.67 0.67 0.3; visual box size=0.67 0.67 0.3
- added link set1_arm2, mass 1.0; collision box size=0.67 0.67 0.3; visual box size=0.67 0.67 0.3
- added link set2_arm1, mass 1.0; collision box size=0.67 0.67 0.3; visual box size=0.67 0.67 0.3
- added link set2_arm2, mass 1.0; collision box size=0.67 0.67 0.3; visual box size=0.67 0.67 0.3
- added link set3_arm1, mass 1.0; collision box size=0.67 0.67 0.3; visual box size=0.67 0.67 0.3
- added link set3_arm2, mass 1.0; collision box size=0.67 0.67 0.3; visual box size=0.67 0.67 0.3
- added link set4_arm1, mass 1.0; collision box size=0.67 0.67 0.3; visual box size=0.67 0.67 0.3
- added link set4_arm2, mass 1.0; collision box size=0.67 0.67 0.3; visual box size=0.67 0.67 0.3
Joints:
- removed joint arm_0_joint1
- removed joint arm_0_jointBase
- removed joint arm_1_joint1
- removed joint arm_1_jointBase
- removed joint arm_2_joint1
- removed joint arm_2_jointBase
- removed joint arm_3_joint1
- removed joint arm_3_jointBase
- added joint set1_joint1: type revolute, parent set1_arm1, child set1_arm2, origin xyz=0.0 0.68 0.0 rpy=0.0 0.0 0.0, axis 1. 0. 0., limit lower=-1.57 upper=1.57 effort=1.57 velocity=1.57
- added joint set1_jointBase: type fixed, parent base_link, child set1_arm1, origin xyz=0.0 0.34 0.0 rpy=0.0 0.0 0.0, axis 1. 0. 0., limit lower=-1.57 upper=1.57 effort=1.57 velocity=1.57
- added joint set2_joint1: type revolute, parent set2_arm1, child set2_arm2, origin xyz=0.0 0.68 0.0 rpy=0.0 0.0 0.0, axis 1. 0. 0., limit lower=-1.57 upper=1.57 effort=1.57 velocity=1.57
- added joint set2_jointBase: type fixed, parent base_link, child set2_arm1, origin xyz=0.0 -0.34 0.0 rpy=0.0 0.0 3.141, axis 1. 0. 0., limit lower=-1.57 upper=1.57 effort=1.57 velocity=1.57
- added joint set3_joint1: type revolute, parent set3_arm1, child set3_arm2, origin xyz=0.0 0.68 0.0 rpy=0.0 0.0 0.0, axis 1. 0. 0., limit lower=-1.57 upper=1.57 effort=1.57 velocity=1.57
- added joint set3_jointBase: type fixed, parent base_link, child set3_arm1, origin xyz=0.34 0.0 0.0 rpy=0.0 0.0 -1.57, axis 1. 0. 0., limit lower=-1.57 upper=1.57 effort=1.57 velocity=1.57
- added joint set4_joint1: type revolute, parent set4_arm1, child set4_arm2, origin xyz=0.0 0.68 0.0 rpy=0.0 0.0 0.0, axis 1. 0. 0., limit lower=-1.57 upper=1.57 effort=1.57 velocity=1.57
- added joint set4_jointBase: type fixed, parent base_link, child set4_arm1, origin xyz=-0.34 0.0 0.0 rpy=0.0 0.0 1.57, axis 1. 0. 0., limit lower=-1.57 upper=1.57 effort=1.57 velocity=1.57
