Commit message: Added Permutation generation

File: self_estimation/Models/Model_98.urdf (robot description, URDF)
Before this commit: robot Model_0, 9 links, 8 joints
Joints:
- joint arm_0_jointBase: origin xyz=-0.34 0.34 0.0 rpy=0.0 0.0 2.83 -> xyz=0.34 0.0 0.0 rpy=0.0 0.0 -1.31
- joint arm_1_jointBase: origin xyz=0.34 -0.34 0.0 rpy=0.0 0.0 -0.08 -> xyz=-0.34 -0.34 0.0 rpy=0.0 0.0 0.35
- joint arm_2_jointBase: origin xyz=0.34 0.34 0.0 rpy=0.0 0.0 2.71 -> xyz=-0.34 0.0 0.0 rpy=0.0 0.0 1.38
- joint arm_3_jointBase: origin xyz=-0.34 -0.34 0.0 rpy=0.0 0.0 0.21 -> xyz=0.34 0.34 0.0 rpy=0.0 0.0 2.22
