Commit message: bug fixes and more movement generated

File: self_estimation/Models/Model_834.urdf (robot description, URDF)
Before this commit: robot Model_98, 9 links, 8 joints
Joints:
- joint arm_0_jointBase: origin xyz=0.34 0.0 0.0 rpy=0.0 0.0 -1.31 -> xyz=0.0 0.34 0.0 rpy=0.0 0.0 -0.02
- joint arm_1_jointBase: origin xyz=-0.34 -0.34 0.0 rpy=0.0 0.0 0.35 -> xyz=0.0 -0.34 0.0 rpy=0.0 0.0 2.41
- joint arm_2_jointBase: origin xyz=-0.34 0.0 0.0 rpy=0.0 0.0 1.38 -> xyz=0.34 0.0 0.0 rpy=0.0 0.0 -1.21
- joint arm_3_jointBase: origin xyz=0.34 0.34 0.0 rpy=0.0 0.0 2.22 -> xyz=-0.34 -0.34 0.0 rpy=0.0 0.0 0.83
