Commit message: more complex configs

File: self_estimation/Models/testPiece.urdf (robot description, URDF)
Before this commit: robot estimationBasic, 11 links, 10 joints
Joints:
- joint set0_jointBase: origin xyz=0.0 -0.34 0.0 rpy=0.0 0.0 3.140996777702981 -> xyz=0.0 0.34 0.0 rpy=0.0 0.0 -0.3227299089599105
- joint set1_jointBase: origin xyz=-0.34 0.34 0.0 rpy=0.0 0.0 0.9982080703103466 -> xyz=0.34 -0.34 0.0 rpy=0.0 0.0 -2.8242980257441768
- joint set2_jointBase: origin xyz=0.34 0.34 0.0 rpy=0.0 0.0 -1.0760221271669443 -> xyz=-0.34 0.0 0.0 rpy=0.0 0.0 1.5712921478626276
- joint set3_jointBase: origin xyz=0.34 0.34 0.0 rpy=0.0 0.0 -1.0006509717523158 -> xyz=0.0 0.68 0.0 rpy=0.0 0.0 0.0; parent base_link -> set2_arm2
- joint set4_jointBase: origin xyz=-0.34 0.34 0.0 rpy=0.0 0.0 1.0755915533719016 -> xyz=0.34 0.0 0.0 rpy=0.0 0.0 -1.5697355063773173

File: self_estimation/christanRobotLONG.urdf (robot description, URDF)
Before this commit: robot rob, 13 links, 12 joints
Links:
- removed link set6_arm1
- removed link set6_arm2
Joints:
- removed joint set6_joint1
- removed joint set6_jointBase
- joint set3_jointBase: parent set1_arm2 -> set4_arm2
